File: csi.kicad_sch (KiCad schematic)
At the start: 65 parts, among them J7 Conn_FFC_WE_68715014522, J8 Conn_FFC_WE_68715014522, U24 AP22615A_TSOT26, U25 AP22615A_TSOT26, U26 PI4MSD5V9548AZDEX, U27 AP22615A_TSOT26, U28 AP22615A_TSOT26, U31 NTS0102_XSON, U32 NTS0102_XSON

Commit message: Schematic complete. Partial routing
Parts:
- removed C90, C91: C_100n_0402, antmicro-footprints:C_0402_1005Metric, symbol antmicroCapacitors0402:C_100n_0402
- removed C94, C95, C98, C99: C_1u_0402, antmicro-footprints:C_0402_1005Metric, symbol antmicroCapacitors0402:C_1u_0402
- removed D18, D20, D24, D25: LED_G_0603_LTST-C190GKT, antmicro-footprints:LED_0603_1608Metric_G, symbol antmicroLEDIndicationDiscrete:LED_G_0603_LTST-C190GKT
- removed J7, J8: Conn_FFC_WE_68715014522, antmicro-footprints:Conn_FFC_WE_68715014x22, symbol antmicroFCCConnectors:Conn_FFC_WE_68715014522
- removed R10, R9: R_4k7_0402, antmicro-footprints:R_0402_1005Metric, symbol antmicroResistors0402:R_4k7_0402
- removed R103, R107, R108, R122, R50, R51: R_4x0R_0201_array, antmicro-footprints:R_Array_4x0201_Panasonic_EXB18V, symbol antmicroResistorNetworksArrays:R_4x0R_0201_array
- removed R132, R133: R_200R_0402, antmicro-footprints:R_0402_1005Metric, symbol antmicroResistors0402:R_200R_0402
- removed R166, R171, R174, R179: R_0R_0402, antmicro-footprints:R_0402_1005Metric, symbol antmicroResistors0402:R_0R_0402
- removed R180: R_100k_0402, antmicro-footprints:R_0402_1005Metric, symbol antmicroResistors0402:R_100k_0402
- removed R194: R_10k_0402, antmicro-footprints:R_0402_1005Metric, symbol antmicroResistors0402:R_10k_0402
- removed R197, R206: R_470R_0402, antmicro-footprints:R_0402_1005Metric, symbol antmicroResistors0402:R_470R_0402
- removed R36, R48: R_4x2k2_0201_array, antmicro-footprints:R_Array_4x0201_Panasonic_EXB18V, symbol antmicroResistorNetworksArrays:R_4x2k2_0201_array
- removed U27, U28: AP22615A_TSOT26, antmicro-footprints:TSOT23-6, symbol antmicroPMICPowerDistributionSwitchesLoadDrivers:AP22615A_TSOT26
- added C47, C79: C_100n_0603, Capacitor_SMD:C_0603_1608Metric, symbol antmicroCapacitors0402:C_100n_0402
- added D14, D15, D16, D17: LED_G_0603_LTST-C190GKT, LED_SMD:LED_0603_1608Metric, symbol antmicroLEDIndicationDiscrete:LED_G_0603_LTST-C190GKT
- added J1, J16, J6, J9: Conn_01x15_MountingPin, Connector_FFC-FPC:Molex_200528-0150_1x15-1MP_P1.00mm_Horizontal, symbol Connector_Generic_MountingPin:Conn_01x15_MountingPin
- added R10, R2, R51: R_100k_0603, Resistor_SMD:R_0603_1608Metric, symbol antmicroResistors0402:R_100k_0402
- added R101, R102, R26, R36, R48, R54, R55, R63: 2K2, Resistor_SMD:R_0402_1005Metric, symbol Device:R_Small
- added R3, R40, R50, R64, R9: R_10k_0603, Resistor_SMD:R_0603_1608Metric, symbol antmicroResistors0402:R_10k_0402
- added R85, R86, R87, R88, R89, R90: R_4k7_0603, Resistor_SMD:R_0603_1608Metric, symbol antmicroResistors0402:R_4k7_0402
- added U3, U7: AP22615A_TSOT26, Package_TO_SOT_SMD:TSOT-23-6, symbol antmicroPMICPowerDistributionSwitchesLoadDrivers:AP22615A_TSOT26
- C100, C101, C43, C89, C96, C97: value C_100n_0402 -> C_100n_0603; footprint antmicro-footprints:C_0402_1005Metric -> Capacitor_SMD:C_0603_1608Metric
- C39: renamed from C42; value C_100n_0402 -> C_100n_0603; footprint antmicro-footprints:C_0402_1005Metric -> Capacitor_SMD:C_0603_1608Metric
- R161, R162, R167, R168: footprint antmicro-footprints:R_0402_1005Metric -> Resistor_SMD:R_0402_1005Metric
- R163, R193, R66, R67: value R_10k_0402 -> R_10k_0603; footprint antmicro-footprints:R_0402_1005Metric -> Resistor_SMD:R_0603_1608Metric
- R6: value R_100k_0402 -> R_100k_0603; footprint antmicro-footprints:R_0402_1005Metric -> Resistor_SMD:R_0603_1608Metric
- R7, R8: value R_4k7_0402 -> R_4k7_0603; footprint antmicro-footprints:R_0402_1005Metric -> Resistor_SMD:R_0603_1608Metric
- TP36, TP37, TP38, TP39, TP40, TP41, TP42, TP43: footprint antmicro-footprints:TP_SMD_0.75mm -> JetsonCarrier:TP_SMD_0.75mm
- U24, U25: footprint antmicro-footprints:TSOT23-6 -> Package_TO_SOT_SMD:TSOT-23-6
- U26: footprint antmicro-footprints:VQFN-24-1EP_3.8x3.8x1.0mm_P0.5mm -> JetsonCarrier:VQFN-24-1EP_3.8x3.8x1.0mm_P0.5mm
- U31, U32: footprint antmicro-footprints:XSON-8_1x1.95mm_P0.5mm -> JetsonCarrier:XSON-8_1x1.95mm_P0.5mm
Connections:
- net +5V is gone; now on net +3V3: C39.1, U24.6 (IN)
- net +1V8: now also R193.2, R66.1, R67.1, R3.1, R40.2, R50.2, R64.1, R9.2
- net +3V3: now also C47.1, C79.1, R101.1, R102.1, R26.1, R36.1, R48.1, R54.1, R55.1, R63.1, U3.6 (IN), U7.6 (IN); no longer R193.2, R66.1, R67.1
- net CSI0_CLK_N: now also J1.8 (Pin_8)
- net CSI0_CLK_P: now also J1.7 (Pin_7)
- net CSI0_D0_N: now also J1.14 (Pin_14)
- net CSI0_D0_P: now also J1.13 (Pin_13)
- net CSI0_D1_N: now also J1.11 (Pin_11)
- net CSI0_D1_P: now also J1.10 (Pin_10)
- net CSI1_CLK_N: now also J6.8 (Pin_8)
- net CSI1_CLK_P: now also J6.7 (Pin_7)
- net CSI1_D0_N: now also J6.14 (Pin_14)
- net CSI1_D0_P: now also J6.13 (Pin_13)
- net CSI1_D1_N: now also J6.11 (Pin_11)
- net CSI1_D1_P: now also J6.10 (Pin_10)
- net CSI2_CLK_N: now also J9.8 (Pin_8)
- net CSI2_CLK_P: now also J9.7 (Pin_7)
- net CSI2_D0_N: now also J9.14 (Pin_14)
- net CSI2_D0_P: now also J9.13 (Pin_13)
- net CSI2_D1_N: now also J9.11 (Pin_11)
- net CSI2_D1_P: now also J9.10 (Pin_10)
- net CSI3_CLK_N: now also J16.8 (Pin_8)
- net CSI3_CLK_P: now also J16.7 (Pin_7)
- net CSI3_D0_N: now also J16.14 (Pin_14)
- net CSI3_D0_P: now also J16.13 (Pin_13)
- net CSI3_D1_N: now also J16.11 (Pin_11)
- net CSI3_D1_P: now also J16.10 (Pin_10)
- net GND: now also U26.25 (EP), C47.2, C79.2, D14.1 (C), D15.1 (C), D16.1 (C), D17.1 (C), J1.12 (Pin_12), J1.15 (Pin_15), J1.6 (Pin_6), J1.9 (Pin_9), J1.MP (MountPin), J16.12 (Pin_12), J16.15 (Pin_15), J16.6 (Pin_6), J16.9 (Pin_9), J16.MP (MountPin), J6.12 (Pin_12), J6.15 (Pin_15), J6.6 (Pin_6), J6.9 (Pin_9), J6.MP (MountPin), J9.12 (Pin_12), J9.15 (Pin_15), J9.6 (Pin_6), J9.9 (Pin_9), J9.MP (MountPin), R10.1, R2.1, R51.1, R85.1, R86.1, U3.2 (GND), U7.2 (GND)
- net SCL_CAM0: now also J1.3 (Pin_3), R54.2
- net SCL_CAM1: now also J6.3 (Pin_3), R48.2
- net SCL_CAM2: now also J9.3 (Pin_3), R26.2
- net SCL_CAM3: now also J16.3 (Pin_3), R101.2
- net SDA_CAM0: now also J1.2 (Pin_2), R63.2
- net SDA_CAM1: now also J6.2 (Pin_2), R36.2
- net SDA_CAM2: now also J9.2 (Pin_2), R55.2
- net SDA_CAM3: now also J16.2 (Pin_2), R102.2
- net VSYNC_CAM0: now also U31.4 (A_{2}); no longer U31.5 (A_{1})
- net VSYNC_CAM0_3V3: now also U31.1 (B_{2}), J1.5 (Pin_5); no longer U31.8 (B_{1})
- net VSYNC_CAM1: now also U31.5 (A_{1}); no longer U31.4 (A_{2})
- net VSYNC_CAM1_3V3: now also U31.8 (B_{1}), J6.5 (Pin_5); no longer U31.1 (B_{2})
- net VSYNC_CAM2: now also U32.4 (A_{2}); no longer U32.5 (A_{1})
- net VSYNC_CAM2_3V3: now also U32.1 (B_{2}), J9.5 (Pin_5); no longer U32.8 (B_{1})
- net VSYNC_CAM3: now also U32.5 (A_{1}); no longer U32.4 (A_{2})
- net VSYNC_CAM3_3V3: now also U32.8 (B_{1}), J16.5 (Pin_5); no longer U32.1 (B_{2})
- net CSIA_3V3 renamed 3V3_CAM1
- net 3V3_CAM1: now also J6.1 (Pin_1), R90.1
- net CSIA_3V3_ISET renamed 3V3_CAM1_ISET
- net CSIA_5V renamed 3V3_CAM0
- net 3V3_CAM0: now also J1.1 (Pin_1), R89.1
- net CSIA_5V_ISET renamed 3V3_CAM0_ISET
- net CSIA_FLG renamed CAM0_FLG
- net CAM0_FLG: no longer U25.3 (FLG)
- net CSIA_PEN renamed CAM0_PEN
- net CAM0_PEN: now also R2.2; no longer R6.2, U25.4 (EN)
- net CSIB_FLG renamed CAM3_FLG
- net CAM3_FLG: now also U7.3 (FLG)
- new net: D15.2 (A), R88.2
- new net: D14.2 (A), R87.2
- new net: D17.2 (A), R90.2
- new net: D16.2 (A), R89.2
- new net 3V3_CAM2: J9.1 (Pin_1), R88.1, U3.1 (OUT)
- new net 3V3_CAM2_ISET: R85.2, U3.5 (ISET)
- new net 3V3_CAM3: J16.1 (Pin_1), R87.1, U7.1 (OUT)
- new net 3V3_CAM3_ISET: R86.2, U7.5 (ISET)
- new net CAM1_FLG: R3.2, U25.3 (FLG)
- new net CAM1_PEN: R40.1, R6.2, U25.4 (EN)
- new net CAM2_FLG: R64.2, U3.3 (FLG)
- new net CAM2_PEN: R10.2, R9.1, U3.4 (EN)
- new net CAM3_PEN: R50.1, R51.2, U7.4 (EN)
- new net MCLK_CAM0: J1.4 (Pin_4)
- new net MCLK_CAM1: J6.4 (Pin_4)
- new net MCLK_CAM2: J9.4 (Pin_4)
- new net MCLK_CAM3: J16.4 (Pin_4)
- no-connect marks 37 -> 0
Other:
- note added: "CSI connectors"
- note removed: "AVAILABLE CSI CONFIGURATIONS:"
- note removed: "CONNECTOR J7"
- note removed: "CONNECTOR J8"
- note removed: "CSI Mux"
- note removed: "CSI connector J7"
- note removed: "CSI connector J8"
- note removed: "CSI0 x2"
- note removed: "CSI0 x4"
- note removed: "CSI0x2 CSI2x2"
- note removed: "CSI0x2 CSI2x4"
- note removed: "CSI0x4 CSI2x2"
- note removed: "CSI0x4 CSI2x4"
- note removed: "CSI1 x2"
- note removed: "CSI1x2"
- note removed: "CSI2 x2"
- note removed: "CSI2 x4"
- note removed: "CSI3 x2"
- note removed: "CSI3x2"
- note removed: "CSI3x2 CSI1x2"
- note removed: "NONE"
- note removed: "TO CONNECTOR J7"
- note removed: "TO CONNECTOR J8"
- company: Antmicro Ltd -> Argus-1 Cubesat
- title: Jetson Orin Baseboard -> Jetson Carrier Board
- moved on the sheet: C100, C101, C39, C43, C89, C97, R161, R162, R163, R167, R168, R193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
