File: jetson-orin-baseboard.kicad_sch (KiCad schematic)
At the start: 4 parts

Commit message: Schematic complete. Partial routing
Parts:
- H3, H4, H5, H6: value Spacer_Drill3.7mm_H6.5mm_9774065151R -> MountingHole_Pad; footprint antmicro-footprints:Spacer_Drill3.7mm_H6.5mm_9774065151R -> mainboard:MountingHole2; Author Antmicro -> (none); DNI (none) -> DNI; License Apache-2.0 -> (none); Manufacturer Würth Elektronik -> (none)
Other:
- sheet USB Debug, DP renamed USB Debug, USB2
- sheet USB3 renamed USB3, Recovery
- removed sheet Ethernet
- added sheet USB3-2 (usb3-2.kicad_sch)
- note removed: "Jetson Orin Baseboard"
- note removed: "github.com/antmicro/jetson-orin-baseboard"
- company: Antmicro Ltd -> Argus-1 Cubesat
- title: Jetson Orin Baseboard -> Jetson Carrier Board
- moved on the sheet: H3, H4, H5, H6
