File: m-2.kicad_sch (KiCad schematic)
At the start: 61 parts, among them J1 Bus_M.2_2199230-6, J2 Bus_M.2_1-2199230-6, M3 Mech_M2_2280_H2.5mm, U2 74LVC2G07_SOT457, U3 74LVC2G07_SOT457, Y1 Oscillator_32.768kHz_ECS_2520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

Commit message: Schematic complete. Partial routing
Parts:
- removed A2: Mech_M2_2242_H2.5mm, antmicro-footprints:Mech_M2_2242_H2.5mm, symbol antmicroModules:Mech_M2_2242_H2.5mm
- removed C10, C9: C_220n_0402, antmicro-footprints:C_0402_1005Metric, symbol antmicroCapacitors0402:C_220n_0402
- removed C11, C12: C_10u_0603, antmicro-footprints:C_0603_1608Metric, symbol antmicroCapacitors0603:C_10u_0603
- removed C7, C8: C_100n_0402, antmicro-footprints:C_0402_1005Metric, symbol antmicroCapacitors0402:C_100n_0402
- removed D51, D52: LED_G_0603_LTST-C190GKT, antmicro-footprints:LED_0603_1608Metric_G, symbol antmicroLEDIndicationDiscrete:LED_G_0603_LTST-C190GKT
- removed J1: Bus_M.2_2199230-6, antmicro-footprints:Bus_M.2_Socket_Key_E_TE_2199230-6, symbol antmicroPciConnectors:Bus_M.2_2199230-6
- removed R14, R15, R16, R17, R18, R20, R29, R30, R31, R52: R_0R_0402, antmicro-footprints:R_0402_1005Metric, symbol antmicroResistors0402:R_0R_0402
- removed R186, R187: R_200R_0402, antmicro-footprints:R_0402_1005Metric, symbol antmicroResistors0402:R_200R_0402
- removed R21, R22: R_4x0R_0201_array, antmicro-footprints:R_Array_4x0201_Panasonic_EXB18V, symbol antmicroResistorNetworksArrays:R_4x0R_0201_array
- removed R27, R28, R32: R_47k_0402, antmicro-footprints:R_0402_1005Metric, symbol antmicroResistors0402:R_47k_0402
- removed SP7: Spacer_H2.5mm_9774025151, antmicro-footprints:Spacer_Drill3.7mm_H2.5mm_9774025151R, symbol antmicroMechanicalParts:Spacer_Drill3.7mm_H2.5mm_9774025151R
- removed TP6, TP7, TP8, TP9: TP_0.75mm_SMD, antmicro-footprints:TP_SMD_0.75mm, symbol antmicroTestPoints:TP_0.75mm_SMD
- removed U2, U3: 74LVC2G07_SOT457, antmicro-footprints:SC-74-6_1.5x2.9mm_P0.95mm, symbol antmicroLogicBuffersDriversReceiversTransceivers:74LVC2G07_SOT457
- C13, C14, C15, C16, C17, C18, C19, C20: footprint antmicro-footprints:C_0402_1005Metric -> Capacitor_SMD:C_0402_1005Metric
- C21, C22, C23, C24: footprint antmicro-footprints:C_0603_1608Metric -> Capacitor_SMD:C_0603_1608Metric
- C25: value C_100n_0402 -> C_100n_0603; footprint antmicro-footprints:C_0402_1005Metric -> Capacitor_SMD:C_0603_1608Metric
- D1: footprint antmicro-footprints:LED_0603_1608Metric_G -> LED_SMD:LED_0603_1608Metric
- J2: footprint antmicro-footprints:Bus_M.2_Socket_Key_M_TE_1-2199230-6 -> JetsonCarrier:Bus_M.2_Socket_Key_M_TE_1-2199230-6
- M3: footprint antmicro-footprints:Mech_M2_2280_H2.5mm -> JetsonCarrier:Mech_M2_2280_H2.5mm
- R13, R19, R37, R38: footprint antmicro-footprints:R_0402_1005Metric -> Resistor_SMD:R_0402_1005Metric
- R143: footprint antmicro-footprints:R_0603_1608Metric -> Resistor_SMD:R_0603_1608Metric
- R39: value R_200R_0402 -> R_200R_0603; footprint antmicro-footprints:R_0402_1005Metric -> Resistor_SMD:R_0603_1608Metric
- SP8: footprint antmicro-footprints:Spacer_Drill3.7mm_H2.5mm_9774025151R -> JetsonCarrier:Spacer_Drill3.7mm_H2.5mm_9774025151R
- TP10, TP11, TP12: footprint antmicro-footprints:TP_SMD_0.75mm -> JetsonCarrier:TP_SMD_0.75mm
- Y1: footprint antmicro-footprints:Oscillator_SMD_ECS_2520MV_2.5x2mm -> JetsonCarrier:Oscillator_SMD_ECS_2520MV_2.5x2mm
Connections:
- net ~{M2_M_CLKREQ0} is gone; now on net PCIE0_CLKREQ*: J2.52 (~{CLKREQ}), R38.2
- net ~{M2_M_PERST} is gone; now on net PCIE0_RST*: J2.50 (~{PERST}), R37.2
- net ~{M2_M_PEWAKE0} is gone; now on net PCIE_WAKE_SEL0: J2.54 (~{PEWAKE})
- no-connect marks 23 -> 0
Other:
- note removed: "BT"
- note removed: "NOTE about PCIe 0 role switching: For details, refer to the PCIe section of "Jeton Orin NX Series Product Design Guide" https://developer.nvidia.com/jetson-orin-nx-series-design-guide"
- note removed: "NOTE: DNP for M.2 key M endpoint role"
- note removed: "NOTE: DNP for M.2 key M root port role"
- note removed: "PCIe0 Root Port / Endpoint mode selector"
- note removed: "PCIe1 1x1 key E"
- note removed: "WLAN"
- company: Antmicro Ltd -> Argus-1 Cubesat
- title: Jetson Orin Baseboard -> Jetson Carrier Board
- moved on the sheet: C13, C14, C15, C16, C17, C18, C19, C20, C21, C22, C23, C24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
