File: peripherals.kicad_sch (KiCad schematic)
At the start: 93 parts, among them J10 Molex_PicoBlade_1x4_0533980471, J11 ERF8-040-05.0-L-DV-K-TR, J14 JST_SH_1x4_SM04B-SRSS-TB-LF-SN, J9 Tag-Connect_TC2050-IDC-NL_2x5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, Q10 PJE138K, Q9 PJE138K, U30 TPD4E05U06QDQARQ1, U33 NTS0102_XSON, U34 PCAL6408A_VQFN, U35 AP22653_DFN

Commit message: Schematic complete. Partial routing
Parts:
- removed C104, C111, C113: C_100n_0402, antmicro-footprints:C_0402_1005Metric, symbol antmicroCapacitors0402:C_100n_0402
- removed C105, C106, C107, C114, C115: C_1u_0402, antmicro-footprints:C_0402_1005Metric, symbol antmicroCapacitors0402:C_1u_0402
- removed C108, C109, C110, C112: C_220n_0402, antmicro-footprints:C_0402_1005Metric, symbol antmicroCapacitors0402:C_220n_0402
- removed D16, D17, D19, D21, D22, D23, D39, D40, D41, D42, D43, D44, D45, D46, D47, D48, D49, D50, D58, D59: TPD1E0B04_XDFN-2, antmicro-footprints:XDFN-2_1x0.60mm, symbol antmicroTVSDiodes:TPD1E0B04_XDFN-2
- removed D26, D27, D54: LED_G_0603_LTST-C190GKT, antmicro-footprints:LED_0603_1608Metric_G, symbol antmicroLEDIndicationDiscrete:LED_G_0603_LTST-C190GKT
- removed J11: ERF8-040-05.0-L-DV-K-TR, antmicro-footprints:Conn_Socket_Samtec_ERF8_2x40_ERF8-040-05.0-L-DV-K-TR, symbol antmicroB2BConnectors:Socket_Samtec_ERF8_2x40_ERF8-040-05.0-L-DV-K-TR
- removed J9: Tag-Connect_TC2050-IDC-NL_2x5_P1.27mm, antmicro-footprints:Tag-Connect_TC2050-IDC-NL_2x5_P1.27mm, symbol antmicroTestPoints:Tag-Connect_TC2050-IDC-NL_2x5_P1.27mm
- removed Q10, Q9: PJE138K, antmicro-footprints:SOT-523, symbol antmicroTransistorsFETsMOSFETsSingle:PJE138K
- removed R100, R101, R102, R26, R54, R63, R64: R_4x330R_0402_array, antmicro-footprints:R_Array_4x0402, symbol antmicroResistorNetworksArrays:R_4x330R_0402_array
- removed R111, R112, R120, R121, R134, R141, R215, R216, R217, R218, R55, R62: R_0R_0402, antmicro-footprints:R_0402_1005Metric, symbol antmicroResistors0402:R_0R_0402
- removed R191, R223, R231: R_200R_0402, antmicro-footprints:R_0402_1005Metric, symbol antmicroResistors0402:R_200R_0402
- removed R195, R204, R25: R_4x0R_0201_array, antmicro-footprints:R_Array_4x0201_Panasonic_EXB18V, symbol antmicroResistorNetworksArrays:R_4x0R_0201_array
- removed R219, R232, R242: R_10k_0402, antmicro-footprints:R_0402_1005Metric, symbol antmicroResistors0402:R_10k_0402
- removed R222, R230: R_100k_0402, antmicro-footprints:R_0402_1005Metric, symbol antmicroResistors0402:R_100k_0402
- removed R233, R235, R248: R_0R_22.4A_0603, antmicro-footprints:R_0603_1608Metric, symbol antmicroResistors0603:R_0R_22.4A_0603
- removed R234, R247: R_0R_0603, antmicro-footprints:R_0603_1608Metric, symbol antmicroResistors0603:R_0R_0603
- removed R335, R336: R_470R_0402, antmicro-footprints:R_0402_1005Metric, symbol antmicroResistors0402:R_470R_0402
- removed S2, S3: SW_SPST_KMR211NGLFS, antmicro-footprints:SW_KMR211NGLFS_SMD, symbol antmicroPushbuttonSwitches:SW_KMR211NGLFS_SMD
- removed U30: TPD4E05U06QDQARQ1, antmicro-footprints:USON-10_2.5x1mm_P0.5mm, symbol antmicroTVSDiodes:TPD4E05U06QDQARQ1
- removed U34: PCAL6408A_VQFN, antmicro-footprints:VQFN-16-1EP_3x3mm_P0.5mm_EP1.68x1.68mm, symbol antmicroInterfaceIOExpanders:PCAL6408A_VQFN
- added C12, C33, C40, C41: C_1u_0603, Capacitor_SMD:C_0603_1608Metric, symbol antmicroCapacitors0402:C_1u_0402
- added J7, J8: Conn_01x10_MountingPin, Connector_FFC-FPC:Molex_200528-0100_1x10-1MP_P1.00mm_Horizontal, symbol Connector_Generic_MountingPin:Conn_01x10_MountingPin
- added U9: SN74AXC4T774, Package_DFN_QFN:UQFN-16_1.8x2.6mm_P0.4mm, symbol JetsonCarrier:SN74AXC4T774
- C130, C44, C48: value C_100n_0402 -> C_100n_0603; footprint antmicro-footprints:C_0402_1005Metric -> Capacitor_SMD:C_0603_1608Metric
- D56, D57: value TPD1E0B04_XDFN-2 -> TPD1E0B04; footprint antmicro-footprints:XDFN-2_1x0.60mm -> Diode_SMD:D_SOD-882
- J10: footprint antmicro-footprints:Conn_Molex_PicoBlade_1x4_0533980471 -> Connector_Molex:Molex_PicoBlade_53398-0471_1x04-1MP_P1.25mm_Vertical; symbol antmicroWire2BoardConnectors:Molex_PicoBlade_1x4_0533980471 -> Connector_Generic_MountingPin:Conn_01x04_MountingPin
- J14: footprint antmicro-footprints:Conn_JST_SH_1x4_SM04B-SRSS-TB-LF-SN -> JetsonCarrier:Conn_JST_SH_1x4_SM04B-SRSS-TB-LF-SN
- R189: value R_10k_0402 -> R_10k_0603; footprint antmicro-footprints:R_0402_1005Metric -> Resistor_SMD:R_0603_1608Metric
- R190: value R_15k_0402 -> R_15k_0603; footprint antmicro-footprints:R_0402_1005Metric -> Resistor_SMD:R_0603_1608Metric
- R192: value R_100k_0402 -> R_100k_0603; footprint antmicro-footprints:R_0402_1005Metric -> Resistor_SMD:R_0603_1608Metric
- R53: value R_4x330R_0402_array -> R_4x0R_0402_array; footprint antmicro-footprints:R_Array_4x0402 -> Resistor_SMD:R_Array_Concave_4x0402; Val R_4x330R_0402 -> R_4x0R
- U33: footprint antmicro-footprints:XSON-8_1x1.95mm_P0.5mm -> JetsonCarrier:XSON-8_1x1.95mm_P0.5mm
- U35: footprint antmicro-footprints:DFN-6-1EP_2x2mm_P0.65mm_EP1x1.6mm -> JetsonCarrier:DFN-6-1EP_2x2mm_P0.65mm_EP1x1.6mm
Connections:
- net GPIO09 is gone; now on net UART1_TXD_CONN: R53.7 (R2.2)
- net GPIO09_CONN is gone; now on net UART1_TXD: R53.2 (R2.1)
- net +1V8: now also C41.2, U9.13 (V_{CCB})
- net +5V: now also C12.2, J7.1 (Pin_1), J7.2 (Pin_2), J7.3 (Pin_3), J7.4 (Pin_4)
- net FAN_PWM: now also U33.4 (A_{2}); no longer U33.5 (A_{1})
- net FAN_PWM_5V: now also U33.1 (B_{2}); no longer U33.8 (B_{1})
- net FAN_TACH: now also U33.5 (A_{1}); no longer U33.4 (A_{2})
- net FAN_TACH_5V: now also U33.8 (B_{1}); no longer U33.1 (B_{2})
- net GND: now also J10.MP (MountPin), C12.1, C33.1, C40.1, C41.1, J7.10 (Pin_10), J7.5 (Pin_5), J7.6 (Pin_6), J7.7 (Pin_7), J7.MP (MountPin), J8.10 (Pin_10), J8.5 (Pin_5), J8.MP (MountPin), U9.6 (DIR4), U9.7 (~{OE}), U9.8 (GND)
- net SPIO_MISO: now also U9.9 (B4)
- net SPIO_MOSI: now also U9.11 (B2)
- net SPIO_SCK: now also U9.10 (B3)
- net UART1_RXD: now also R53.1 (R1.1); no longer R53.8 (R1.2)
- net UART1_RXD_CONN: now also R53.8 (R1.2); no longer R53.1 (R1.1)
- net USB1_D_N: now also J7.9 (Pin_9)
- net USB1_D_P: now also J7.8 (Pin_8)
- net ~{SPI0_CS0}: now also U9.12 (B1)
- new net JETSON_EN: J8.4 (Pin_4)
- new net MB_3V3: C33.2, C40.2, J8.1 (Pin_1), U9.14 (V_{CCA}), U9.15 (DIR1), U9.16 (DIR2), U9.5 (DIR3)
- new net MB_CS: J8.6 (Pin_6), U9.1 (A1)
- new net MB_MISO: J8.9 (Pin_9), U9.4 (A4)
- new net MB_MOSI: J8.7 (Pin_7), U9.2 (A2)
- new net MB_SCK: J8.8 (Pin_8), U9.3 (A3)
- new net MB_SCL: J8.3 (Pin_3)
- new net MB_SDA: J8.2 (Pin_2)
- no-connect marks 15 -> 5
Other:
- note removed: "Buttons"
- note removed: "Debug connector"
- note removed: "Depends on the power source PoE will supply 12 V USB PD will supply 9 V or 15 V For the Nano Fit DC IN we specify 9-15 V"
- note removed: "GPIO expander"
- note removed: "LED indicators"
- note removed: "LOW POWER ONLY FOR LEVEL SHIFTERS"
- note removed: "pinout compatible with www.github.com/antmicro/ftdi-toolkit"
- company: Antmicro Ltd -> Argus-1 Cubesat
- title: Jetson Orin Baseboard -> Jetson Carrier Board
- moved on the sheet: C130, C44, C48, D56, D57, J14, R189, R190, R192, R53, U33, U35
