File: peripherals.kicad_sch (KiCad schematic)
At the start: 20 parts, among them J10 Molex_PicoBlade_1x4_0533980471, J14 JST_SH_1x4_SM04B-SRSS-TB-LF-SN, J7 Conn_01x10_MountingPin, J8 Conn_01x10_MountingPin, U33 NTS0102_XSON, U35 AP22653_DFN, U9 SN74AXC4T774

Commit message: Schematic Cleanup, Complete routing
Parts:
- added TP2, TP29, TP3, TP30, TP31: TP_0.75mm_SMD, JetsonCarrier:TP_SMD_0.75mm, symbol Connector:TestPoint
- C108: renamed from C130; value C_100n_0603 -> 100nF; symbol antmicroCapacitors0402:C_100n_0402 -> Device:C_Small
- C12, C33: value C_1u_0603 -> 1uF; symbol antmicroCapacitors0402:C_1u_0402 -> Device:C_Small
- C40, C41: value C_1u_0603 -> 100nF; symbol antmicroCapacitors0402:C_1u_0402 -> Device:C_Small
- C44, C48: value C_100n_0603 -> 100nF; symbol antmicroCapacitors0402:C_100n_0402 -> Device:C_Small
- D17: renamed from D56; symbol antmicroTVSDiodes:TPD1E0B04_XDFN-2 -> Device:D_TVS_Small
- D18: renamed from D57; symbol antmicroTVSDiodes:TPD1E0B04_XDFN-2 -> Device:D_TVS_Small
- J10: value Molex_PicoBlade_1x4_0533980471 -> 0533980471
- J14: value JST_SH_1x4_SM04B-SRSS-TB-LF-SN -> SM04B-SRSS-TB-LF-SN; symbol antmicroWire2BoardConnectors:JST_SH_1x4_SM04B-SRSS-TB-LF-SN -> JetsonCarrier:JST_SH_1x4_SM04B-SRSS-TB-LF-SN
- J7, J8: value Conn_01x10_MountingPin -> 200528-0100
- R145: renamed from R189; value R_10k_0603 -> 10k; symbol antmicroResistors0402:R_10k_0402 -> Device:R_Small
- R146: renamed from R192; value R_100k_0603 -> 100k; symbol antmicroResistors0402:R_100k_0402 -> Device:R_Small; now in the parts list
- R147: renamed from R190; value R_15k_0603 -> 15k; symbol antmicroResistors0402:R_15k_0402 -> Device:R_Small
- RN3: renamed from R53; value R_4x0R_0402_array -> 4x0R; symbol antmicroResistorNetworksArrays:R_4x330R_0402_array -> Device:R_Pack04
- U33: value NTS0102_XSON -> NTS0102; symbol antmicroLogicTranslatorsLevelShifters:NTS0102_XSON -> JetsonCarrier:NTS0102
- U35: value AP22653_DFN -> AP22653; symbol antmicroPMICPowerDistributionSwitchesLoadDrivers:AP22653_DFN -> JetsonCarrier:AP22653
Connections:
- net +1V8: now also C41.1, C44.1; no longer C41.2, C44.2
- net +3V3: now also C108.2, R145.1; no longer C108.1, R145.2
- net +5V: now also C48.1; no longer C48.2
- net GND: now also C108.1, C41.2, C44.2, C48.2, R146.2, R147.2; no longer C108.2, C41.1, C44.1, C48.1, R146.1, R147.1
- net I2C_CONN_PEN: now also R145.2, R146.1; no longer R145.1, R146.2
- net UART1_RXD: now also RN3.3 (R3.1); no longer RN3.1 (R1.1)
- net UART1_RXD_CONN: now also RN3.6 (R3.2), TP2.1; no longer RN3.8 (R1.2)
- net UART1_TXD: now also RN3.4 (R4.1); no longer RN3.2 (R2.1)
- net UART1_TXD_CONN: now also RN3.5 (R4.2), TP3.1; no longer RN3.7 (R2.2)
- net at U35.2 (ISET): now also R147.1; no longer R147.2
- new net JETSON_RST: TP31.1
- new net SLEEP/~{WAKE}: TP29.1
- new net ~{MOD_SLEEP}: TP30.1
Other:
- note removed: "Expansion connector"
- note removed: "Expansion connector resistors"
- moved on the sheet: C108, C12, C33, C40, C41, C44, C48, D18, J7, J8, R145, R146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
