File: som.kicad_sch (KiCad schematic)
At the start: 34 parts, among them J15 Bus_DDR4_SODIMM_CUSTOM_Jetson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, M1 Jetson-Orin-NX-Nano, U4 NTS0102_XSON

Commit message: Schematic complete. Partial routing
Parts:
- removed H1, H2: Spacer_Drill3.7mm_H6.5mm_9774065151R, antmicro-footprints:Spacer_Drill3.7mm_H6.5mm_9774065151R, symbol antmicroMechanicalParts:Spacer_Drill3.7mm_H6.5mm_9774065151R
- removed R1, R2, R3: R_0R_0402, antmicro-footprints:R_0402_1005Metric, symbol antmicroResistors0402:R_0R_0402
- removed TP2, TP3, TP4, TP5: TP_0.75mm_SMD, antmicro-footprints:TP_SMD_0.75mm, symbol antmicroTestPoints:TP_0.75mm_SMD
- added R31: R_200k_0603, Resistor_SMD:R_0402_1005Metric, symbol antmicroResistors0402:R_4k7_0402
- added R84, R92, R93, R94, R95, R96, R97, R98: R_0R_0402, Resistor_SMD:R_0402_1005Metric, symbol antmicroResistors0402:R_0R_0402
- BT1: footprint antmicro-footprints:MS621FE-FL11E -> JetsonCarrier:MS621FE-FL11E
- C1, C2, C3, C4, C46: footprint antmicro-footprints:C_0603_1608Metric -> Capacitor_SMD:C_0603_1608Metric
- C35: renamed from C38; footprint antmicro-footprints:C_0603_1608Metric -> Capacitor_SMD:C_0603_1608Metric
- C36: renamed from C39; footprint antmicro-footprints:C_0603_1608Metric -> Capacitor_SMD:C_0603_1608Metric
- C37: renamed from C40; value C_100n_0402 -> C_100n_0603; footprint antmicro-footprints:C_0402_1005Metric -> Capacitor_SMD:C_0603_1608Metric
- C38: renamed from C41; value C_100n_0402 -> C_100n_0603; footprint antmicro-footprints:C_0402_1005Metric -> Capacitor_SMD:C_0603_1608Metric
- D34: footprint antmicro-footprints:SOD-523 -> Diode_SMD:D_SOD-523
- D55: value TPD1E0B04_XDFN-2 -> TPD1E0B04; footprint antmicro-footprints:XDFN-2_1x0.60mm -> Diode_SMD:D_SOD-882; MPN TPD1E0B04DPYR -> TPD1E0B04
- FB1: footprint antmicro-footprints:FB_1206_3216Metric -> Inductor_SMD:L_1206_3216Metric
- J15: footprint antmicro-footprints:TE_2309413 -> JetsonCarrier:TE_2309413
- M1: footprint antmicro-footprints:Module_Jetson-Orin-NX-Nano -> JetsonCarrier:Module_Jetson-Orin-NX-Nano
- R11, R12, R294: footprint antmicro-footprints:R_0402_1005Metric -> Resistor_SMD:R_0402_1005Metric
- R4, R5: footprint antmicro-footprints:R_0402_1005Metric -> Resistor_SMD:R_0402_1005Metric; DNP DNP -> (none); now fitted
- R80: value R_4k7_0402 -> R_200k_0603; footprint antmicro-footprints:R_0402_1005Metric -> Resistor_SMD:R_0402_1005Metric; Val 4k7 -> 200k
- S1: value SW_SPST_KMR211NGLFS -> KMR211NGLFS; footprint antmicro-footprints:SW_KMR211NGLFS_SMD -> Button_Switch_SMD:SW_Push_1P1T-SH_NO_CK_KMR2xxG; symbol antmicroPushbuttonSwitches:SW_KMR211NGLFS_SMD -> JetsonCarrier:SW_KMR211NGLFS_SMD
- TP35, TP44: footprint antmicro-footprints:TP_SMD_0.75mm -> JetsonCarrier:TP_SMD_0.75mm
- U4: footprint antmicro-footprints:XSON-8_1x1.95mm_P0.5mm -> JetsonCarrier:XSON-8_1x1.95mm_P0.5mm
Connections:
- net +1V8: now also R80.1, R31.2; no longer R80.2
- net DEBUG_RXD: now also U4.1 (B_{2}); no longer U4.8 (B_{1})
- net DEBUG_RXD_1V8: now also U4.4 (A_{2}); no longer U4.5 (A_{1})
- net DEBUG_TXD: now also U4.8 (B_{1}); no longer U4.1 (B_{2})
- net DEBUG_TXD_1V8: now also U4.5 (A_{1}); no longer U4.4 (A_{2})
- net GND: now also J15.261 (MP), J15.262 (MP), S1.SH
- net MCLK_CAM1: now reaches J15.122 (CAM1_MCLK)
- net MCLK_CAM0: now reaches J15.116 (CAM0_MCLK)
- net USBC0_PEN: now reaches J15.124 (GPIO02)
- net GBE_LED_ACT: no longer names the net of J15.194 (GBE_LED_ACT)
- net GBE_LED_LINK: no longer names the net of J15.188 (GBE_LED_LINK)
- net GBE_MDI0_N: no longer names the net of J15.184 (GBE_MDI0_N)
- net GBE_MDI0_P: no longer names the net of J15.186 (GBE_MDI0_P)
- net GBE_MDI1_N: no longer names the net of J15.190 (GBE_MDI1_N)
- net GBE_MDI1_P: no longer names the net of J15.192 (GBE_MDI1_P)
- net GBE_MDI2_N: no longer names the net of J15.196 (GBE_MDI2_N)
- net GBE_MDI2_P: no longer names the net of J15.198 (GBE_MDI2_P)
- net GBE_MDI3_N: no longer names the net of J15.202 (GBE_MDI3_N)
- net GBE_MDI3_P: no longer names the net of J15.204 (GBE_MDI3_P)
- net GPIO01 renamed MCLK_CAM2
- net GPIO010 renamed ~{USBC1_INT}
- net ~{USBC1_INT}: now also R80.2; no longer R80.1
- net GPIO07: no longer names the net of J15.206 (GPIO07/PWM)
- net GPIO09 renamed ~{USBC0_INT}
- net ~{USBC0_INT}: now also R31.1
- net GPIO11 renamed MCLK_CAM3
- net I2C2_SCL: no longer names the net of J15.232 (I2C2_SCL)
- net I2C2_SDA: no longer names the net of J15.234 (I2C2_SDA)
- net I2S0_LRCK: no longer names the net of J15.197 (I2S0_FS)
- net I2S0_LRCK: now also R94.1
- net I2S0_SCLK: no longer names the net of J15.199 (I2S0_SCLK)
- net I2S0_SCLK: now also R84.1
- net I2S0_SDIN: no longer names the net of J15.195 (I2S0_DIN)
- net I2S0_SDIN: now also R93.1
- net I2S0_SDOUT: no longer names the net of J15.193 (I2S0_DOUT)
- net I2S0_SDOUT: now also R92.1
- net I2S1_LRCK: no longer names the net of J15.224 (I2S1_FS)
- net I2S1_LRCK: now also R98.1
- net I2S1_SCLK: no longer names the net of J15.226 (I2S1_SCLK)
- net I2S1_SCLK: now also R95.1
- net I2S1_SDIN: no longer names the net of J15.222 (I2S1_DIN)
- net I2S1_SDIN: now also R97.1
- net I2S1_SDOUT: no longer names the net of J15.220 (I2S1_DOUT)
- net I2S1_SDOUT: now also R96.1
- net PCIE1_CLKREQ*: no longer names the net of J15.182 (~{PCIE1_CLKREQ})
- net PCIE1_CLK_N: no longer names the net of J15.173 (PCIE1_CLK_N)
- net PCIE1_CLK_P: no longer names the net of J15.175 (PCIE1_CLK_P)
- net PCIE1_RST*: no longer names the net of J15.183 (~{PCIE1_RST})
- net PCIE1_RX0_N: no longer names the net of J15.167 (PCIE1_RX0_N)
- net PCIE1_RX0_P: no longer names the net of J15.169 (PCIE1_RX0_P)
- net PCIE1_TX0_N: no longer names the net of J15.172 (PCIE1_TX0_N)
- net PCIE1_TX0_P: no longer names the net of J15.174 (PCIE1_TX0_P)
- net PCIE2_CLKREQ*: no longer names the net of J15.221 (~{PCIE2_CLKREQ})
- net PCIE2_CLK_N: no longer names the net of J15.52 (PCIE2_CLK_N)
- net PCIE2_CLK_P: no longer names the net of J15.54 (PCIE2_CLK_P)
- net PCIE2_RST*: no longer names the net of J15.219 (~{PCIE2_RST})
- net PCIE2_RX0_N: no longer names the net of J15.40 (PCIE2_RX0_N)
- net PCIE2_RX0_P: no longer names the net of J15.42 (PCIE2_RX0_P)
- net PCIE2_RX1_N: no longer names the net of J15.58 (PCIE3_RX0_N)
- net PCIE2_RX1_P: no longer names the net of J15.60 (PCIE3_RX0_P)
- net PCIE2_TX0_N: no longer names the net of J15.46 (PCIE2_TX0_N)
- net PCIE2_TX0_P: no longer names the net of J15.48 (PCIE2_TX0_P)
- net PCIE2_TX1_N: no longer names the net of J15.64 (PCIE3_TX0_N)
- net PCIE2_TX1_P: no longer names the net of J15.66 (PCIE3_TX0_P)
- net PCIE3_CLKREQ*: no longer names the net of J15.225 (~{PCIE3_CLKREQ})
- net PCIE3_CLK_N: no longer names the net of J15.227 (PCIE3_CLK_N)
- net PCIE3_CLK_P: no longer names the net of J15.229 (PCIE3_CLK_P)
- net PCIE3_RST*: no longer names the net of J15.223 (~{PCIE3_RST})
- net SPI1_MISO: no longer names the net of J15.108 (SPI1_MISO)
- net SPI1_MOSI: no longer names the net of J15.104 (SPI1_MOSI)
- net SPI1_SCK: no longer names the net of J15.106 (SPI1_SCK)
- net UART0_CTS: no longer names the net of J15.105 (~{UART0_CTS})
- net UART0_RTS: no longer names the net of J15.103 (~{UART0_RTS})
- net UART0_RXD: no longer names the net of J15.101 (UART0_RXD)
- net UART0_TXD: no longer names the net of J15.99 (UART0_TXD)
- net USBSS1_RX_N: no longer names the net of J15.39 (USBSS1_RX_N)
- net USBSS1_RX_P: no longer names the net of J15.41 (USBSS1_RX_P)
- net USBSS1_TX_N: no longer names the net of J15.45 (USBSS1_TX_N)
- net USBSS1_TX_P: no longer names the net of J15.47 (USBSS1_TX_P)
- net USER_BTN0 renamed USBC1_FLG
- net USER_BTN1: no longer names the net of J15.130 (GPIO06)
- net USER_LED0 renamed USBC0_FLG
- net USER_LED1 renamed USBC1_PEN
- net ~{SPI1_CS0}: no longer names the net of J15.110 (~{SPI1_CS0})
- net ~{SPI1_CS1}: no longer names the net of J15.112 (~{SPI1_CS1})
- new net CAM0_FLG: R84.2
- new net CAM0_PEN: R92.2
- new net CAM1_FLG: R93.2
- new net CAM1_PEN: R94.2
- new net CAM2_FLG: R95.2
- new net CAM2_PEN: R96.2
- new net CAM3_FLG: R97.2
- new net CAM3_PEN: R98.2
- no-connect marks 14 -> 63
Other:
- company: Antmicro Ltd -> Argus-1 Cubesat
- title: Jetson Orin Baseboard -> Jetson Carrier Board
- moved on the sheet: C37, C38, D55, J15H, R80, U4
