File: som.kicad_sch (KiCad schematic)
At the start: 34 parts, among them J15 Bus_DDR4_SODIMM_CUSTOM_Jetson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, M1 Jetson-Orin-NX-Nano, U4 NTS0102_XSON

Commit message: Schematic Cleanup, Complete routing
Parts:
- removed M1: Jetson-Orin-NX-Nano, JetsonCarrier:Module_Jetson-Orin-NX-Nano, symbol antmicroModules:Jetson-Orin-NX-Nano
- added H6, H7: 9774065151, JetsonCarrier:Spacer_Drill3.7mm_H2.5mm_9774025151R, symbol Mechanical:MountingHole_Pad
- added TP4: TP_0.75mm_SMD, JetsonCarrier:TP_SMD_0.75mm, symbol Connector:TestPoint
- BT1: value Battery_Holder_MS621FE-FL11E -> MS621FE-FL11E; symbol antmicroBatteryHoldersClipsContacts:Battery_Holder_MS621FE-FL11E -> Device:Battery_Cell
- C1, C2, C3, C35, C36, C4, C46: value C_22u_16V_0603 -> 22uF; symbol antmicroCapacitors0603:C_22u_16V_0603 -> Device:C_Small
- C37, C38: value C_100n_0603 -> 100nF; symbol antmicroCapacitors0402:C_100n_0402 -> Device:C_Small
- D15: renamed from D55; symbol antmicroTVSDiodes:TPD1E0B04_XDFN-2 -> Device:D_TVS_Small
- D21: renamed from D34; symbol antmicroDiodesRectifiersSingle:RB521S30T1G -> Device:D_Schottky
- FB1: value FB_10Z_10A_1206 -> 74279221100; symbol antmicroFerriteBeadsandChips:FB_10Z_10A_WE-MPSB_1206 -> Device:FerriteBead_Small
- J15: symbol antmicroSoMConnectors:Bus_DDR4_SODIMM_CUSTOM_Jetson-Orin-H9.2mm-socket -> JetsonCarrier:Bus_DDR4_SODIMM_CUSTOM_Jetson-Orin-H9.2mm-socket
- R11, R12: value R_0R_0402 -> 0R; symbol antmicroResistors0402:R_0R_0402 -> Device:R_Small
- R174: renamed from R294; value R_2k2_0402 -> 2k2; symbol antmicroResistors0402:R_2k2_0402 -> Device:R_Small
- R31, R80: value R_200k_0603 -> 200k; symbol antmicroResistors0402:R_4k7_0402 -> Device:R_Small
- R4, R5, R84, R92, R93, R94, R95, R96, R97, R98: value R_0R_0402 -> 0R; symbol antmicroResistors0402:R_0R_0402 -> Device:R_Small; now in the parts list
- TP25: renamed from TP35; symbol antmicroTestPoints:TP_0.75mm_SMD -> Connector:TestPoint
- TP7: renamed from TP44; symbol antmicroTestPoints:TP_0.75mm_SMD -> Connector:TestPoint
- U4: value NTS0102_XSON -> NTS0102; symbol antmicroLogicTranslatorsLevelShifters:NTS0102_XSON -> JetsonCarrier:NTS0102
- renumbered S1 to BTN1
Connections:
- net +1V8: now also C37.1, R31.1, R80.2; no longer C37.2, R31.2, R80.1
- net +3V3: now also C38.1; no longer C38.2
- net GND: now also C3.2, C35.2, C36.2, C37.2, C38.2, C4.2, C46.2, H6.1, H7.1; no longer BTN1.4, C3.1, C35.1, C36.1, C37.1, C38.1, C4.1, C46.1
- net PMIC_BBAT: now also R174.1; no longer R174.2
- net SoM_5V_IN: now also C3.1, C35.1, C36.1, C4.1, C46.1; no longer C3.2, C35.2, C36.2, C4.2, C46.2
- net VSYNC_CAM0: now also R12.1; no longer R12.2
- net ~{FORCE_RECOVERY}: no longer BTN1.3
- net ~{USBC0_INT}: now also R31.2; no longer R31.1
- net ~{USBC1_INT}: now also R80.1; no longer R80.2
- net at BT1.1 (+): now also R174.2; no longer R174.1
- net at J15.114 (CAM0_PWDN): now also R12.2; no longer R12.1
- net CAN_RX: no longer names the net of J15.143 (CAN_RX)
- net CAN_TX: no longer names the net of J15.145 (CAN_TX)
- net ~{SPI0_CS1}: no longer names the net of J15.97 (~{SPI0_CS1})
- net ~{SPI0_CS1}: now also TP4.1
- no-connect marks 63 -> 65
Other:
- moved on the sheet: C1, C2, C3, C35, C36, C37, C38, C4, C46, FB1, R11, R12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
