File: supply.kicad_sch (KiCad schematic)
At the start: 106 parts, among them J12 Molex_Nano-Fit_1x2_SMD_105430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, Q11 PJE138K, Q13 BCM857BS-7-F, Q14 BCM857BS-7-F, Q15 SSM3J332R, Q16 SSM3J332R, Q18 SSM3J332R, Q5 PJE138K, Q6 SSM3J332R, Q7 PJE138K, Q8 PJE138K, SW1 SW_SPDT_PCM12SMTR, U1 TPS56C230, U29 TPS56C230, U37 74LVC2G14_SOT457, U38 74LVC1G175_SOT457, U41 NCP730BMT330_WSON, U42 TPS7A0518P_SOT23-5

Commit message: Schematic complete. Partial routing
Parts:
- removed C150: C_1u_16V_0402, antmicro-footprints:C_0402_1005Metric, symbol antmicroCapacitors0402:C_1u_16V_0402
- removed C50: C_100n_0402, antmicro-footprints:C_0402_1005Metric, symbol antmicroCapacitors0402:C_100n_0402
- removed D29: DF2S30FS_SOD, antmicro-footprints:SOD-923, symbol antmicroTVSDiodes:DF2S30FS_SOD
- removed J12: Molex_Nano-Fit_1x2_SMD_1054301202, antmicro-footprints:Conn_Molex_Nano-Fit_1x2_SMD_1054301202, symbol antmicroWire2BoardConnectors:Molex_Nano-Fit_1x2_SMD_1054301202
- removed Q13, Q14: BCM857BS-7-F, antmicro-footprints:SOT-363, symbol antmicroTransistorsBipolarArrays:BCM857BS-7-F
- removed Q15, Q16, Q18: SSM3J332R, antmicro-footprints:SOT-23-3, symbol antmicroTransistorsFETsMOSFETsSingle:SSM3J332R
- removed Q7: PJE138K, antmicro-footprints:SOT-523, symbol antmicroTransistorsFETsMOSFETsSingle:PJE138K
- removed R164, R165: R_4k7_0402, antmicro-footprints:R_0402_1005Metric, symbol antmicroResistors0402:R_4k7_0402
- removed R175, R252, R253: R_0R_22.4A_0603, antmicro-footprints:R_0603_1608Metric, symbol antmicroResistors0603:R_0R_22.4A_0603
- removed R249: R_100k_0402, antmicro-footprints:R_0402_1005Metric, symbol antmicroResistors0402:R_100k_0402
- removed R250, R251, R254, R255: R_10k_0402, antmicro-footprints:R_0402_1005Metric, symbol antmicroResistors0402:R_10k_0402
- removed R263: R_0R_0402, antmicro-footprints:R_0402_1005Metric, symbol antmicroResistors0402:R_0R_0402
- removed TP14, TP23: TP_0.75mm_SMD, antmicro-footprints:TP_SMD_0.75mm, symbol antmicroTestPoints:TP_0.75mm_SMD
- added C26: C_3300p_0603, Capacitor_SMD:C_0603_1608Metric, symbol Device:C_Small
- added C28, C30: C_10n_0603, Capacitor_SMD:C_0603_1608Metric, symbol Device:C
- added J11: Conn_01x04, JetsonCarrier:TE_282834-4, symbol Connector_Generic:Conn_01x04
- added Q1, Q9: BSS138DWQ-7, Package_TO_SOT_SMD:SOT-363_SC-70-6, symbol Mainboard:BSS138DWQ-7
- added Q10, Q7: MBT2222ADW1T1, Package_TO_SOT_SMD:SOT-363_SC-70-6, symbol Transistor_BJT:MBT2222ADW1T1
- added R1: ?R, Resistor_SMD:R_2512_6332Metric, symbol Device:R_Small
- added R25: R_1k_0603, Resistor_SMD:R_0603_1608Metric, symbol Device:R_Small
- added R59, R75: R_680R_0603, Resistor_SMD:R_0603_1608Metric, symbol Device:R_Small
- added R65, R76: R_100k_0603, Resistor_SMD:R_0603_1608Metric, symbol Device:R_Small
- added R68, R69, R77, R78: R_10k_0603, Resistor_SMD:R_0603_1608Metric, symbol Device:R_Small
- added R70, R79: R_200k_0603, Resistor_SMD:R_0603_1608Metric, symbol Device:R_Small
- added R71, R74: R_0R_0603, Resistor_SMD:R_0603_1608Metric, symbol Device:R_Small
- added R81: R_10k_0603, Resistor_SMD:R_0603_1608Metric, symbol antmicroResistors0402:R_200k_0402
- added R82: R_10k_0603, Resistor_SMD:R_0603_1608Metric, symbol antmicroResistors0402:R_10k_0402
- added U6: ADM1176-1ARMZ-R7, Package_SO:MSOP-10_3x3mm_P0.5mm, symbol Mainboard:ADM1176-1ARMZ-R7
- C102, C118, C119, C122, C124, C125, C6: value C_100n_0402 -> C_100n_0603; footprint antmicro-footprints:C_0402_1005Metric -> Capacitor_SMD:C_0603_1608Metric
- C103, C120, C126, C127, C128, C129, C134, C153, C154: footprint antmicro-footprints:C_0603_1608Metric -> Capacitor_SMD:C_0603_1608Metric
- C116, C117, C137, C83: value C_10u_0402 -> C_10u_0603; footprint antmicro-footprints:C_0402_1005Metric -> Capacitor_SMD:C_0603_1608Metric
- C121, C151, C152, C5: footprint antmicro-footprints:C_0805_2012Metric -> Capacitor_SMD:C_0805_2012Metric
- C123, C142, C93: value C_1u_0402 -> C_1u_0603; footprint antmicro-footprints:C_0402_1005Metric -> Capacitor_SMD:C_0603_1608Metric
- D28, D30, D31, D32, D33: footprint antmicro-footprints:SOD-923 -> Diode_SMD:D_SOD-923
- D36, D37: footprint antmicro-footprints:SOD-523 -> Diode_SMD:D_SOD-523
- D53: footprint antmicro-footprints:LED_0603_1608Metric_G -> LED_SMD:LED_0603_1608Metric
- D60, D61: value TPD1E0B04_XDFN-2 -> TPD1E0B04; footprint antmicro-footprints:XDFN-2_1x0.60mm -> Diode_SMD:D_SOD-882
- L1, L2: footprint antmicro-footprints:L_Coilcraft-XAL6030 -> Inductor_SMD:L_Coilcraft_XAL6030-XXX
- Q11, Q5, Q8: footprint antmicro-footprints:SOT-523 -> Package_TO_SOT_SMD:SOT-523
- Q6: footprint antmicro-footprints:SOT-23-3 -> Package_TO_SOT_SMD:SOT-23-3
- R159, R173, R181, R188, R239, R240, R259: value R_10k_0402 -> R_10k_0603; footprint antmicro-footprints:R_0402_1005Metric -> Resistor_SMD:R_0603_1608Metric
- R169: value R_110k_0402 -> R_110k_0603; footprint antmicro-footprints:R_0402_1005Metric -> Resistor_SMD:R_0603_1608Metric
- R170: value R_15k_0402 -> R_15k_0603; footprint antmicro-footprints:R_0402_1005Metric -> Resistor_SMD:R_0603_1608Metric
- R172, R178, R182: value R_0R_22.4A_0603 -> R_0R_22.4A_0805; footprint antmicro-footprints:R_0603_1608Metric -> Resistor_SMD:R_0805_2012Metric
- R176: value R_90k9_0402 -> R_90k9_0603; footprint antmicro-footprints:R_0402_1005Metric -> Resistor_SMD:R_0603_1608Metric
- R177: value R_20k_0402 -> R_20k_0603; footprint antmicro-footprints:R_0402_1005Metric -> Resistor_SMD:R_0603_1608Metric
- R183: footprint antmicro-footprints:R_0402_1005Metric -> Resistor_SMD:R_0402_1005Metric
- R236: value R_200R_0402 -> R_200R_0603; footprint antmicro-footprints:R_0402_1005Metric -> Resistor_SMD:R_0603_1608Metric
- R237, R238: value R_220k_0402 -> R_220k_0603; footprint antmicro-footprints:R_0402_1005Metric -> Resistor_SMD:R_0603_1608Metric
- R256: value R_1k_0402 -> R_10k_0603; footprint antmicro-footprints:R_0402_1005Metric -> Resistor_SMD:R_0603_1608Metric; Val 1k -> 10k
- R257: footprint antmicro-footprints:R_0402_1005Metric -> Resistor_SMD:R_0603_1608Metric
- R258, R261: value R_200k_0402 -> R_200k_0603; footprint antmicro-footprints:R_0402_1005Metric -> Resistor_SMD:R_0603_1608Metric
- R260, R264, R268: value R_0R_0402 -> R_0R_0603; footprint antmicro-footprints:R_0402_1005Metric -> Resistor_SMD:R_0603_1608Metric
- R273, R276: footprint antmicro-footprints:R_0603_1608Metric -> Resistor_SMD:R_0603_1608Metric
- S4, S5: value SW_SPST_KMR211NGLFS -> KMR211NGLFS; footprint antmicro-footprints:SW_KMR211NGLFS_SMD -> Button_Switch_SMD:SW_Push_1P1T-SH_NO_CK_KMR2xxG; symbol antmicroPushbuttonSwitches:SW_KMR211NGLFS_SMD -> JetsonCarrier:SW_KMR211NGLFS_SMD
- SW1: footprint antmicro-footprints:PCM12SMTR -> Button_Switch_SMD:SW_SPDT_PCM12
- TP52, TP53, TP54, TP55: footprint antmicro-footprints:TP_SMD_0.75mm -> JetsonCarrier:TP_SMD_0.75mm
- U1, U29: footprint antmicro-footprints:QFN-20-1EP_3x3mm_P0.45mm -> JetsonCarrier:QFN-20-1EP_3x3mm_P0.45mm
- U37, U38: footprint antmicro-footprints:SOT-23-6 -> Package_TO_SOT_SMD:SOT-23-6
- U41: footprint antmicro-footprints:WSON-6-1EP_2x2mm_P0.65mm -> JetsonCarrier:WSON-6-1EP_2x2mm_P0.65mm
- U42: footprint antmicro-footprints:SOT-23-5 -> Package_TO_SOT_SMD:SOT-23-5
Connections:
- net 3V3_STDB: now also R82.2
- net 5V0_EN: now also R82.1
- net GND: now also S4.SH, S5.SH, C26.1, C28.2, C30.2, J11.2 (Pin_2), J11.4 (Pin_4), Q1.1 (S2), Q1.4 (S1), Q9.1 (S2), Q9.4 (S1), U6.4 (GND)
- net VCC: now also R1.1, R25.1, U6.2 (SENSE); no longer R188.2
- net VBATT: now reaches D28.1
- net VBATT: now also R188.2, J11.1 (Pin_1), J11.3 (Pin_3), R1.2, U6.1 (VCC)
- net JETSON_EN: now reaches C116.2, D36.2, D60.2, R258.1, S4.1, S4.3, SW1.3, U37.1
- net at C124.2, D61.2, Q8.1 (G)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: now also R81.1
- new net: Q9.2 (G2), Q9.3 (D2), R76.2
- new net: Q10.5 (B2), Q9.6 (D1), R75.2, R77.2
- new net: C30.1, Q9.5 (G1), R79.2
- new net: Q1.2 (G2), Q1.3 (D2), R65.2
- new net: C28.1, Q1.5 (G1), R70.2
- new net: Q10.2 (B1), R75.1
- new net: R25.2, U6.3 (ON)
- new net: Q7.2 (B1), R59.1
- new net: Q1.6 (D1), Q7.5 (B2), R59.2, R68.2
- new net: C26.2, U6.5 (TIMER)
- new net JETSON_RST: R81.2
- new net MB_3V3: R65.1, R68.1, R69.1, R76.1, R77.1, R78.1
- new net MB_SCL: Q7.1 (E1), Q7.3 (C2), R71.1
- new net MB_SDA: Q10.1 (E1), Q10.3 (C2), R74.1
- new net PWR_SCL: Q7.4 (E2), Q7.6 (C1), R69.2, R70.1, R71.2, U6.6 (SCL)
- new net PWR_SDA: Q10.4 (E2), Q10.6 (C1), R74.2, R78.2, R79.1, U6.7 (SDA)
- no-connect marks 3 -> 4
Other:
- note added: "6.4-8.4V"
- note added: "I2C Bus Protection - Power Monitor & USB Charger"
- note added: "I2C1 ADDR"
- note removed: "9-15V"
- note removed: "INPUT SELECTOR AND SOFT START"
- note removed: "PD CONTROLLER HAS IDEAL DIODE BUILT-IN"
- company: Antmicro Ltd -> Argus-1 Cubesat
- title: Jetson Orin Baseboard -> Jetson Carrier Board
- moved on the sheet: C116, C117, C118, C119, C124, D28, D32, D36, D37, D53, D60, D61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
