File: supply.kicad_sch (KiCad schematic)
At the start: 108 parts, among them J11 Conn_01x04, Q1 BSS138DWQ-7, Q10 MBT2222ADW1T1, Q11 PJE138K, Q5 PJE138K, Q6 SSM3J332R, Q7 MBT2222ADW1T1, Q8 PJE138K, Q9 BSS138DWQ-7, SW1 SW_SPDT_PCM12SMTR, U1 TPS56C230, U29 TPS56C230, U37 74LVC2G14_SOT457, U38 74LVC1G175_SOT457, U41 NCP730BMT330_WSON, U42 TPS7A0518P_SOT23-5, U6 ADM1176-1ARMZ-R7

Commit message: Schematic Cleanup, Complete routing
Parts:
- added R62, R91: 150k, Resistor_SMD:R_0603_1608Metric, symbol Device:R_Small
- C102, C6: value C_100n_0603 -> 100nF; symbol antmicroCapacitors0402:C_100n_0402 -> Device:C_Small
- C103: renamed from C124; value C_100n_0603 -> 100nF; symbol antmicroCapacitors0402:C_100n_0402 -> Device:C_Small
- C104: renamed from C125; value C_100n_0603 -> 100nF; symbol antmicroCapacitors0402:C_100n_0402 -> Device:C_Small
- C105: renamed from C134; value C_10u_25V_0603 -> 10uF; symbol antmicroCapacitors0603:C_10u_25V_0603 -> Device:C_Small
- C106: renamed from C137; value C_10u_0603 -> 10uF; symbol antmicroCapacitors0402:C_10u_0402 -> Device:C_Small
- C107: renamed from C142; value C_1u_0603 -> 1uF; symbol antmicroCapacitors0402:C_1u_0402 -> Device:C_Small
- C26: value C_3300p_0603 -> 3300pF
- C28, C30: value C_10n_0603 -> 10nF; symbol Device:C -> Device:C_Small
- C5: value C_22u_25V_0805 -> 22uF; symbol antmicroCapacitorsmisc:C_22u_25V_0805 -> Device:C_Small
- C53: renamed from C116; value C_10u_0603 -> 10uF; symbol antmicroCapacitors0402:C_10u_0402 -> Device:C_Small
- C54: renamed from C117; value C_10u_0603 -> 10uF; symbol antmicroCapacitors0402:C_10u_0402 -> Device:C_Small
- C55: renamed from C118; value C_100n_0603 -> 100nF; symbol antmicroCapacitors0402:C_100n_0402 -> Device:C_Small
- C56: renamed from C119; value C_100n_0603 -> 100nF; symbol antmicroCapacitors0402:C_100n_0402 -> Device:C_Small
- C58: renamed from C151; value C_22u_25V_0805 -> 22uF; symbol antmicroCapacitorsmisc:C_22u_25V_0805 -> Device:C_Small
- C59: renamed from C152; value C_22u_25V_0805 -> 22uF; symbol antmicroCapacitorsmisc:C_22u_25V_0805 -> Device:C_Small
- C65: renamed from C121; value C_22u_25V_0805 -> 22uF; symbol antmicroCapacitorsmisc:C_22u_25V_0805 -> Device:C_Small
- C76: renamed from C122; value C_100n_0603 -> 100nF; symbol antmicroCapacitors0402:C_100n_0402 -> Device:C_Small
- C77: renamed from C123; value C_1u_0603 -> 1uF; symbol antmicroCapacitors0402:C_1u_0402 -> Device:C_Small; Val 1u -> 1uF
- C78: renamed from C126; value C_22u_16V_0603 -> 22uF; symbol antmicroCapacitors0603:C_22u_16V_0603 -> Device:C_Small
- C80: renamed from C103; value C_22u_16V_0603 -> 22uF; symbol antmicroCapacitors0603:C_22u_16V_0603 -> Device:C_Small
- C81: renamed from C127; value C_22u_16V_0603 -> 22uF; symbol antmicroCapacitors0603:C_22u_16V_0603 -> Device:C_Small
- C82: renamed from C129; value C_22u_16V_0603 -> 22uF; symbol antmicroCapacitors0603:C_22u_16V_0603 -> Device:C_Small
- C83: value C_10u_0603 -> 10uF; symbol antmicroCapacitors0402:C_10u_0402 -> Device:C_Small
- C84: renamed from C128; value C_22u_16V_0603 -> 22uF; symbol antmicroCapacitors0603:C_22u_16V_0603 -> Device:C_Small
- C85: renamed from C120; value C_22u_16V_0603 -> 22uF; symbol antmicroCapacitors0603:C_22u_16V_0603 -> Device:C_Small
- C90: renamed from C154; value C_22u_16V_0603 -> 22uF; symbol antmicroCapacitors0603:C_22u_16V_0603 -> Device:C_Small
- C91: renamed from C153; value C_22u_16V_0603 -> 22uF; symbol antmicroCapacitors0603:C_22u_16V_0603 -> Device:C_Small
- C93: value C_1u_0603 -> 1uF; symbol antmicroCapacitors0402:C_1u_0402 -> Device:C_Small
- D14: renamed from D53; symbol antmicroLEDIndicationDiscrete:LED_G_0603_LTST-C190GKT -> Device:LED_Small_Filled
- D16: renamed from D61; symbol antmicroTVSDiodes:TPD1E0B04_XDFN-2 -> Device:D_TVS_Small
- D19: renamed from D60; symbol antmicroTVSDiodes:TPD1E0B04_XDFN-2 -> Device:D_TVS_Small
- D22: renamed from D36; symbol antmicroDiodesRectifiersSingle:RB521S30T1G -> Device:D_Schottky
- D23: renamed from D37; symbol antmicroDiodesRectifiersSingle:RB521S30T1G -> Device:D_Schottky
- D24: renamed from D28; value DF2S30FS_SOD -> VTVS8V5ASMF; footprint Diode_SMD:D_SOD-923 -> Diode_SMD:D_SMF; symbol antmicroTVSDiodes:DF2S30FS_SOD -> Device:D_Zener_Filled
- D25: renamed from D32; symbol antmicroTVSDiodes:ESD9X5.0ST5G -> Device:D_Zener_Filled
- D26: renamed from D33; value ESD9X5.0ST5G -> ESD9X3.3ST5G; symbol antmicroTVSDiodes:ESD9X5.0ST5G -> Device:D_Zener_Filled
- D27: renamed from D30; value ESD9X5.0ST5G -> ESD9X3.3ST5G; symbol antmicroTVSDiodes:ESD9X5.0ST5G -> Device:D_Zener_Filled
- D28: renamed from D31; value ESD9X5.0ST5G -> ESD1V8WT; footprint Diode_SMD:D_SOD-923 -> Diode_SMD:D_SOD-523; symbol antmicroTVSDiodes:ESD9X5.0ST5G -> Device:D_Zener_Filled
- J11: value Conn_01x04 -> 282834-4
- L1, L2: value L_1u8_14A_XAL6030 -> XAL6030-182MEC; symbol antmicroFixedInductors:L_1u8_14A_Coilcraft-XAL6030 -> Device:L_Small
- Q1, Q9: symbol Mainboard:BSS138DWQ-7 -> JetsonCarrier:BSS138DWQ-7
- Q11, Q5, Q8: symbol antmicroTransistorsFETsMOSFETsSingle:PJE138K -> JetsonCarrier:PJE138K
- Q6: symbol antmicroTransistorsFETsMOSFETsSingle:SSM3J332R -> JetsonCarrier:SSM3J332R
- R148: renamed from R188; value R_10k_0603 -> 10k; symbol antmicroResistors0402:R_10k_0402 -> Device:R_Small
- R149: renamed from R256; value R_10k_0603 -> 10k; symbol antmicroResistors0402:R_1k_0402 -> Device:R_Small
- R150: renamed from R257; value R_200k_0402 -> 200k; symbol antmicroResistors0402:R_200k_0402 -> Device:R_Small
- R151: renamed from R258; value R_200k_0603 -> 200k; symbol antmicroResistors0402:R_200k_0402 -> Device:R_Small
- R152: renamed from R236; value R_200R_0603 -> 200R; symbol antmicroResistors0402:R_200R_0402 -> Device:R_Small
- R153: renamed from R261; value R_200k_0603 -> 200k; symbol antmicroResistors0402:R_200k_0402 -> Device:R_Small
- R154: renamed from R259; value R_10k_0603 -> 10k; symbol antmicroResistors0402:R_10k_0402 -> Device:R_Small
- R155: renamed from R260; value R_0R_0603 -> 0R; symbol antmicroResistors0402:R_0R_0402 -> Device:R_Small
- R156: renamed from R237; value R_220k_0603 -> 220k; symbol antmicroResistors0402:R_220k_0402 -> Device:R_Small; now in the parts list
- R157: renamed from R159; value R_10k_0603 -> 10k; symbol antmicroResistors0402:R_10k_0402 -> Device:R_Small
- R158: renamed from R238; value R_220k_0603 -> 220k; symbol antmicroResistors0402:R_220k_0402 -> Device:R_Small; now in the parts list
- R159: renamed from R173; value R_10k_0603 -> 10k; symbol antmicroResistors0402:R_10k_0402 -> Device:R_Small
- R160: renamed from R264; value R_0R_0603 -> 0R; symbol antmicroResistors0402:R_0R_0402 -> Device:R_Small
- R161: renamed from R239; value R_10k_0603 -> 10k; symbol antmicroResistors0402:R_10k_0402 -> Device:R_Small
- R162: renamed from R240; value R_10k_0603 -> 10k; symbol antmicroResistors0402:R_10k_0402 -> Device:R_Small
- R163: renamed from R169; value R_110k_0603 -> 110k; symbol antmicroResistors0402:R_110k_0402 -> Device:R_Small
- R164: renamed from R170; value R_15k_0603 -> 15k; symbol antmicroResistors0402:R_15k_0402 -> Device:R_Small
- R165: renamed from R176; value R_90k9_0603 -> 90k9; symbol antmicroResistors0402:R_90k9_0402 -> Device:R_Small
- R166: renamed from R177; value R_20k_0603 -> 20k; symbol antmicroResistors0402:R_20k_0402 -> Device:R_Small
- R167: renamed from R268; value R_0R_0603 -> 0R; symbol antmicroResistors0402:R_0R_0402 -> Device:R_Small
- R168: renamed from R172; value R_0R_22.4A_0805 -> 0R; symbol antmicroResistors0603:R_0R_22.4A_0603 -> Device:R_Small
- R169: renamed from R178; value R_0R_22.4A_0805 -> 0R; symbol antmicroResistors0603:R_0R_22.4A_0603 -> Device:R_Small
- R170: renamed from R273; value R_0R_0603 -> 0R; symbol antmicroResistors0603:R_0R_0603 -> Device:R_Small
- R171: renamed from R276; value R_0R_0603 -> 0R; symbol antmicroResistors0603:R_0R_0603 -> Device:R_Small
- R172: renamed from R181; value R_10k_0603 -> 10k; symbol antmicroResistors0402:R_10k_0402 -> Device:R_Small
- R173: renamed from R182; value R_0R_22.4A_0805 -> 0R; symbol antmicroResistors0603:R_0R_22.4A_0603 -> Device:R_Small; now in the parts list
- R181: renamed from R183; value R_0R_0402 -> 0R; symbol antmicroResistors0402:R_0R_0402 -> Device:R_Small; now in the parts list
- R25: value R_1k_0603 -> 1k
- R59, R75: value R_680R_0603 -> 680R
- R65, R76: value R_100k_0603 -> 100k
- R68, R69, R77, R78: value R_10k_0603 -> 10k
- R70, R79: value R_200k_0603 -> 200k
- R71, R74: value R_0R_0603 -> 0R
- R81: value R_10k_0603 -> 10k; symbol antmicroResistors0402:R_200k_0402 -> Device:R_Small
- R82: value R_10k_0603 -> 10k; symbol antmicroResistors0402:R_10k_0402 -> Device:R_Small
- SW1: value SW_SPDT_PCM12SMTR -> PCM12SMTR; symbol antmicroSlideSwitches:SW_SPDT_PCM12SMTR -> JetsonCarrier:PCM12SMTR
- TP21: renamed from TP54; symbol antmicroTestPoints:TP_0.75mm_SMD -> Connector:TestPoint
- TP23: renamed from TP52; symbol antmicroTestPoints:TP_0.75mm_SMD -> Connector:TestPoint
- TP24: renamed from TP55; symbol antmicroTestPoints:TP_0.75mm_SMD -> Connector:TestPoint
- TP28: renamed from TP53; symbol antmicroTestPoints:TP_0.75mm_SMD -> Connector:TestPoint
- U1, U29: symbol antmicroDCDCConverters:TPS56C230 -> JetsonCarrier:TPS56C230
- U37: value 74LVC2G14_SOT457 -> 74LVC2G14; symbol antmicroLogicBuffersDriversReceiversTransceivers:74LVC2G14_SOT457 -> JetsonCarrier:74LVC2G14
- U38: value 74LVC1G175_SOT457 -> 74LVC1G175; symbol antmicroLogicGatesandInverters:74LVC1G175_SOT457 -> JetsonCarrier:74LVC1G175
- U41: value NCP730BMT330_WSON -> NCP730BMT330; symbol antmicroPMICVoltageRegulatorsLinear:NCP730BMT330_WSON -> JetsonCarrier:NCP730BMT330
- U42: value TPS7A0518P_SOT23-5 -> TPS7A0518P; symbol antmicroPMICVoltageRegulatorsLinear:TPS7A0518P_SOT23-5 -> JetsonCarrier:TPS7A0518P
- U6: symbol Mainboard:ADM1176-1ARMZ-R7 -> JetsonCarrier:ADM1176-1ARMZ-R7
- renumbered S4 to BTN2, S5 to BTN3
Connections:
- net +1V8: now also R171.1; no longer R171.2
- net 1V8_LDO: now also C107.1, R171.2; no longer C107.2, R171.1
- net 3V3_FB: now also R165.1, R166.1; no longer R165.2, R166.2
- net 3V3_LDO: now also C106.1, R170.2; no longer C106.2, R170.1
- net 3V3_OUT: now also C78.1, C81.1, C84.1, C90.1, R165.2; no longer C78.2, C81.2, C84.2, C90.2, R165.1
- net 3V3_STDB: now also R149.1, R154.1, R170.1; no longer BTN3.3, R149.2, R154.2, R170.2
- net 5V_OUT: now also C80.1, C82.1, C85.1, C91.1, R168.2; no longer C80.2, C82.2, C85.2, C91.2, R168.1
- net 5V_SoM: now also R168.1, R172.1; no longer R168.2, R172.2
- net GND: now also C105.2, C106.2, C107.2, C53.2, C54.2, C58.2, C65.2, C78.2, C80.2, C81.2, C82.2, C84.2, C85.2, C90.2, C91.2, C93.2, R153.2, R159.2, R166.2, R62.2, R91.2; no longer BTN2.4, C105.1, C106.1, C107.1, C53.1, C54.1, C58.1, C65.1, C78.1, C80.1, C81.1, C82.1, C84.1, C85.1, C90.1, C91.1, C93.1, R153.1, R159.1, R166.1
- net JETSON_EN: now also C53.1; no longer BTN2.3, C53.2
- net VBATT: now also R148.1; no longer R148.2
- net VCC: now also C105.1, C58.1, C65.1; no longer C105.2, C58.2, C65.2
- net ~{SHUTDOWN_REQ}: now also R152.1; no longer R152.2
- net at Q11.3 (D), U38.6 (~{CLR}): now also R154.2; no longer R154.1
- net at D14.2 (A): now also R148.2; no longer R148.1
- net at R157.2, U1.15 (MODE): now also R156.2; no longer R156.1
- net at R158.1, U29.15 (MODE): now also R159.1; no longer R159.2
- net at C77.2, R158.2, U29.17 (V_{CC}): now also R162.1; no longer R162.2
- net at R150.1, SW1.2: now also R149.2; no longer R149.1
- net at D22.1 (K), D23.2 (A), R150.2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: now also C54.1; no longer C54.2
- net at U29.9 (PG): now also R162.2; no longer R162.1
- net at R161.1: now also C93.1, R156.1, U1.17 (V_{CC}); no longer U1.9 (PG)
- net at D23.1 (K): now also R152.2; no longer R152.1
- net at BTN3.2, C103.2, D16.2 (A2)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: now also R153.1; no longer BTN3.4, R153.2
- net at Q5.3 (D), Q6.1 (G): now also R172.2; no longer R172.1
- net at U6.8 (A0): now also R62.1
- net at U6.9 (A1): now also R91.1
- new net: R161.2, U1.9 (PG)
Other:
- note removed: "I2C1 ADDR"
- moved on the sheet: C102, C103, C104, C105, C106, C107, C26, C5, C53, C54, C55, C56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
