File: usb.kicad_sch (KiCad schematic)
At the start: 130 parts, among them J3 USB-C_USB4105-GF-A, J4 Conn_USB-C_WE_632723300011, U10 TUSB1046-DCIRNQ, U11 TPD4E05U06QDQARQ1, U12 AP22615A_TSOT26, U13 TPD4E05U06QDQARQ1, U14 TPD4E05U06QDQARQ1, U15 TPD4E05U06QDQARQ1, U16 TPD4E05U06QDQARQ1, U5 FT230X_QFN, U6 TPS65988DHRSHR, U7 W25Q80DV_USON, U8 NCP730BMT330_WSON, U9 AP22615A_TSOT26

Commit message: Schematic complete. Partial routing
Parts:
- removed C136, C148: C_4u7_25V_0402, antmicro-footprints:C_0402_1005Metric, symbol antmicroCapacitors0402:C_4u7_25V_0402
- removed C140, C141, C143, C144, C26, C33, C36, C37, C45, C53, C54, C55, C57, C58, C60, C61, C62, C63, C65: C_100n_0402, antmicro-footprints:C_0402_1005Metric, symbol antmicroCapacitors0402:C_100n_0402
- removed C149: C_1u_16V_0402, antmicro-footprints:C_0402_1005Metric, symbol antmicroCapacitors0402:C_1u_16V_0402
- removed C28, C30, C35, C49, C56, C59: C_10u_0402, antmicro-footprints:C_0402_1005Metric, symbol antmicroCapacitors0402:C_10u_0402
- removed D35: RB521S30T1G, antmicro-footprints:SOD-523, symbol antmicroDiodesRectifiersSingle:RB521S30T1G
- removed D4, D5, D9: LED_G_0603_LTST-C190GKT, antmicro-footprints:LED_0603_1608Metric_G, symbol antmicroLEDIndicationDiscrete:LED_G_0603_LTST-C190GKT
- removed D7: DF2S30FS_SOD, antmicro-footprints:SOD-923, symbol antmicroTVSDiodes:DF2S30FS_SOD
- removed J4: Conn_USB-C_WE_632723300011, antmicro-footprints:USB-C_Receptacle_WE_632723300011, symbol antmicroUSBConnectors:USB-C_WE_632723300011
- removed R104, R78: R_2k2_0402, antmicro-footprints:R_0402_1005Metric, symbol antmicroResistors0402:R_2k2_0402
- removed R106, R130, R246, R262, R81: R_4k7_0402, antmicro-footprints:R_0402_1005Metric, symbol antmicroResistors0402:R_4k7_0402
- removed R109, R110: R_2M_0402, antmicro-footprints:R_0402_1005Metric, symbol antmicroResistors0402:R_2M_0402
- removed R131, R85, R86, R87, R88, R89, R90, R91, R92, R93, R94, R95, R96, R97, R98: R_1k_0402, antmicro-footprints:R_0402_1005Metric, symbol antmicroResistors0402:R_1k_0402
- removed R144, R158, R244, R41, R58, R59, R65, R70, R71, R75, R76, R79, R82, R84: R_0R_0402, antmicro-footprints:R_0402_1005Metric, symbol antmicroResistors0402:R_0R_0402
- removed R205, R207, R43, R45: R_100k_0402, antmicro-footprints:R_0402_1005Metric, symbol antmicroResistors0402:R_100k_0402
- removed R33: R_4x0R_0201_array, antmicro-footprints:R_Array_4x0201_Panasonic_EXB18V, symbol antmicroResistorNetworksArrays:R_4x0R_0201_array
- removed R42, R44, R74, R77, R83, R99: R_10k_0402, antmicro-footprints:R_0402_1005Metric, symbol antmicroResistors0402:R_10k_0402
- removed R68, R69: R_200R_0402, antmicro-footprints:R_0402_1005Metric, symbol antmicroResistors0402:R_200R_0402
- removed TP13, TP18, TP19, TP20, TP24, TP25, TP26, TP27, TP28: TP_0.75mm_SMD, antmicro-footprints:TP_SMD_0.75mm, symbol antmicroTestPoints:TP_0.75mm_SMD
- removed U10: TUSB1046-DCIRNQ, antmicro-footprints:WQFN-40_1EP_6x3mm_Pitch0.4mm_EP4.7x2.7mm, symbol antmicroInterfaceControllers:TUSB1046-DCIRNQ
- removed U12, U9: AP22615A_TSOT26, antmicro-footprints:TSOT23-6, symbol antmicroPMICPowerDistributionSwitchesLoadDrivers:AP22615A_TSOT26
- removed U13, U14, U15, U16: TPD4E05U06QDQARQ1, antmicro-footprints:USON-10_2.5x1mm_P0.5mm, symbol antmicroTVSDiodes:TPD4E05U06QDQARQ1
- removed U6: TPS65988DHRSHR, antmicro-footprints:IC_TPS65987DDHRSHR, symbol antmicroInterfaceControllers:TPS65988DHRSHR
- removed U7: W25Q80DV_USON, antmicro-footprints:USON-8_2x3mm_P0.5mm, symbol antmicroMemory:W25Q80DV_USON
- added R100: R_5K1_0402, Resistor_SMD:R_0402_1005Metric, symbol antmicroResistors0402:R_27R_0402
- added R99: R_5K1_0603, Resistor_SMD:R_0402_1005Metric, symbol antmicroResistors0402:R_27R_0402
- C145, C146: footprint antmicro-footprints:C_0402_1005Metric -> Capacitor_SMD:C_0402_1005Metric
- C147: value C_1u_16V_0402 -> C_1u_16V_0603; footprint antmicro-footprints:C_0402_1005Metric -> Capacitor_SMD:C_0603_1608Metric
- C27, C29, C31, C64: value C_100n_0402 -> C_100n_0603; footprint antmicro-footprints:C_0402_1005Metric -> Capacitor_SMD:C_0603_1608Metric
- C32: footprint antmicro-footprints:C_0603_1608Metric -> Capacitor_SMD:C_0603_1608Metric
- C34: value C_10u_0402 -> C_10u_0603; footprint antmicro-footprints:C_0402_1005Metric -> Capacitor_SMD:C_0603_1608Metric
- D2, D3, D8: footprint antmicro-footprints:LED_0603_1608Metric_G -> LED_SMD:LED_0603_1608Metric
- D6: footprint antmicro-footprints:SOD-923 -> Diode_SMD:D_SOD-923
- J3: footprint antmicro-footprints:USB-C_Receptacle_GCT_USB4105-GF-A -> Connector_USB:USB_C_Receptacle_GCT_USB4105-xx-A_16P_TopMnt_Horizontal
- R105: value R_4k7_0402 -> R_4k7_0603; footprint antmicro-footprints:R_0402_1005Metric -> Resistor_SMD:R_0603_1608Metric
- R117: value R_27R_0402 -> R_27R_0603; footprint antmicro-footprints:R_0402_1005Metric -> Resistor_SMD:R_0603_1608Metric
- R127: value R_27R_0402 -> R_27R_0603; footprint antmicro-footprints:R_0402_1005Metric -> Resistor_SMD:R_0603_1608Metric; Val 27R -> 5K1
- R46: value R_10k_0402 -> R_10k_0603; footprint antmicro-footprints:R_0402_1005Metric -> Resistor_SMD:R_0603_1608Metric
- R56, R57: footprint antmicro-footprints:R_0402_1005Metric -> Resistor_SMD:R_0402_1005Metric
- R72, R73: value R_200R_0402 -> R_200R_0603; footprint antmicro-footprints:R_0402_1005Metric -> Resistor_SMD:R_0603_1608Metric
- TP15, TP16: footprint antmicro-footprints:TP_SMD_0.75mm -> JetsonCarrier:TP_SMD_0.75mm
- U11: footprint antmicro-footprints:USON-10_2.5x1mm_P0.5mm -> JetsonCarrier:USON-10_2.5x1mm_P0.5mm
- U5: footprint antmicro-footprints:QFN-16-1EP_4x4mm_P0.65mm -> JetsonCarrier:QFN-16-1EP_4x4mm_P0.65mm
- U8: footprint antmicro-footprints:WSON-6-1EP_2x2mm_P0.65mm -> JetsonCarrier:WSON-6-1EP_2x2mm_P0.65mm
Connections:
- net GND: now also R100.1, R99.1
- net USBC3_CC1: now also R99.2
- net USBC3_CC2: now also R100.2
- no-connect marks 14 -> 4
Other:
- note removed: "4 LANE DP"
- note removed: "CONFIGURATION"
- note removed: "CTL0"
- note removed: "CTL1"
- note removed: "H"
- note removed: "L"
- note removed: "POWER DOWN"
- note removed: "USB + 2 LANE DP"
- note removed: "USB ONLY"
- note removed: "USB PD Controller"
- note removed: "USB-C 0 Display Port alt mode"
- note removed: "USBC0"
- company: Antmicro Ltd -> Argus-1 Cubesat
- title: Jetson Orin Baseboard -> Jetson Carrier Board
- moved on the sheet: C145, C146, C147, C27, C29, C31, C32, C34, C64, D2, D3, D6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
